File: carte_esp_leds/esp_leds.kicad_sch (KiCad schematic)
At the start: 16 parts, among them J1 LEDs, J2 Prog, J3 USB_B_Mini, SW1 SW_Push, U1 BPC_ESP8266-01_ESP-01, U2 AMS1117-3.3, U3 74AHCT1G125

Commit message: Finalisation
Parts:
- removed J3: USB_B_Mini, Connector_USB:USB_Mini-B_Tensility_54-00023_Vertical, symbol Connector:USB_B_Mini
- added J3: 54819-0519, bpc:BPC_MiniUsb_Molex_54819-0519, symbol bpc:BPC_MiniUsb_Molex_54819-0519
Connections:
- net +5V: now also J3.1 (VBUS), J3.6 (VBUS)
- net GND: now also J3.10 (GND), J3.11 (SHIELD), J3.12 (SHIELD), J3.5 (GND), J3.S1 (SHIELD), J3.S2 (SHIELD)
- new net: J3.2 (D-), J3.7 (D-)
- new net: J3.3 (D+), J3.8 (D+)
- new net: J3.4 (ID), J3.9 (ID)
